Commit message: add mobile base and rgbd sensor

File: plug_description/urdf/mmrobot.urdf.xacro (robot description, xacro)
@@ -1,9 +1,18 @@
 <?xml version="1.0"?>
 <robot name="mmrobot" xmlns:xacro="https://www.ros.org/wiki/xacro" >
+  <xacro:arg name="mu1" default="0.7" />
+  <xacro:arg name="mu2" default="0.98" />
   <xacro:arg name="hardware_interface" default="PositionJointInterface"/>
   <xacro:arg name="robot_name" default="iiwa"/>
   <xacro:arg name="origin_xyz" default="0 0 0"/>
   <xacro:arg name="origin_rpy" default="0 0 0"/>
-  <link name="world"/>
+  <xacro:include filename="$(find plug_description)/urdf/wheelbase.urdf.xacro" />
+  <xacro:wheeler_base_macro>
+    <origin xyz="$(arg origin_xyz)" rpy="$(arg origin_rpy)"/>
+    <xacro:property name="friction_k" value="$(arg mu1)"/>
+    <xacro:property name="friction_s" value="$(arg mu2)"/>
+    <xacro:property name="base_z" value="0.125" />
+    <xacro:property name="bumper_z" value="0.175" />
+  </xacro:wheeler_base_macro>
   <!--iiwa14-->
   <!-- Import Rviz colors -->
@@ -11,16 +20,26 @@
   <!--Import the lbr iiwa macro -->
   <xacro:include filename="$(find iiwa_description)/urdf/iiwa14.xacro"/>
-  <xacro:iiwa14 hardware_interface="$(arg hardware_interface)" robot_name="$(arg robot_name)" parent="world">
-    <origin xyz="$(arg origin_xyz)" rpy="$(arg origin_rpy)" />
+  <xacro:iiwa14 hardware_interface="$(arg hardware_interface)" robot_name="$(arg robot_name)" parent="link_base">
+    <origin xyz="0 0 0.125" rpy="0 0 0" />
   </xacro:iiwa14>
   <!--plug-->
   <xacro:include filename="$(find plug_description)/urdf/plug.urdf.xacro"/>
   <xacro:plug parent="iiwa_link_ee">
-    <origin xyz="-0.011 -0.011 0" rpy="0 0 1.57" />
+    <origin xyz="-0.011 -0.011 0.005" rpy="0 0 1.57" />
   </xacro:plug>
   <!--camera-->
   <xacro:include filename="$(find plug_description)/urdf/camera.urdf.xacro"/>
   <xacro:rpi parent="iiwa_link_ee">
-    <origin xyz="-0.03 0 0.05" rpy="0 -1.57 0" />
+    <origin xyz="-0.01 0 0.062" rpy="0 -1.57 0" />
   </xacro:rpi>
+  <!--RGB-D camera, look forward-->
+  <xacro:include filename="$(find plug_description)/urdf/realsense.urdf.xacro" />
+  <xacro:realsense_macro parent="link_fbumper">
+    <xacro:property name="location_x" value="0.05"/>
+    <xacro:property name="location_y" value="0.0"/>
+    <xacro:property name="location_z" value="0.07"/>
+    <xacro:property name="camera_width" value="640" />
+    <xacro:property name="camera_height" value="480" />
+    <xacro:property name="camera_name" value="rs435" />
+  </xacro:realsense_macro>
 </robot>

File: plug_description/urdf/plug.urdf.xacro (robot description, xacro)
@@ -4,7 +4,29 @@
   <xacro:macro name="plug" params="parent *origin">
     <!--plug-->
+    <joint name="joint_plug_base" type="revolute">
+      <axis xyz="0 0 1" rpy="0 0 0"/>
+      <limit upper="0" lower="0" velocity="0" effort="3.0"/>
+      <dynamics damping="10" friction="1.0"/>
+      <origin xyz="0 0 0" rpy="0 0 0"/>
+      <parent link="${parent}"/>
+      <child link="link_plug_base"/>
+    </joint>
+    <link name="link_plug_base">
+      <visual>
+        <origin rpy="0 0 0" xyz="0 0 0.0025"/>
+        <geometry>
+          <cylinder length="0.005" radius="0.03"/>
+        </geometry>
+      </visual>
+      <collision>
+        <origin rpy="0 0 0" xyz="0 0 0.0025"/>
+        <geometry>
+          <cylinder length="0.005" radius="0.03"/>
+        </geometry>
+      </collision>
+    </link>
     <joint name="joint_plug" type="fixed">
       <xacro:insert_block name="origin"/>
-      <parent link="${parent}"/>
+      <parent link="link_plug_base"/>
       <child link="link_plug"/>
     </joint>
@@ -13,5 +35,5 @@
         <origin rpy="0 0 0" xyz="0 0 0"/>
         <geometry>
-          <mesh filename="package://plug_gazebo/media/materials/obj/plug.obj" scale="0.01 0.01 0.01"/>
+          <mesh filename="package://plug_gazebo/media/materials/obj/plug.obj" scale="1 1 1"/>
         </geometry>
       </visual>
@@ -19,5 +41,5 @@
         <origin rpy="0 0 0" xyz="0 0 0"/>
         <geometry>
-          <mesh filename="package://plug_gazebo/media/materials/obj/plug.obj" scale="0.01 0.01 0.01"/>
+          <mesh filename="package://plug_gazebo/media/materials/obj/plug.obj" scale="1 1 1"/>
         </geometry>
       </collision>

Commit message: add object detection for walloutlet

File: plug_description/urdf/mmrobot.urdf.xacro (robot description, xacro)
@@ -7,5 +7,6 @@
   <xacro:arg name="origin_xyz" default="0 0 0"/>
   <xacro:arg name="origin_rpy" default="0 0 0"/>
-  <xacro:include filename="$(find plug_description)/urdf/wheelbase.urdf.xacro" />
+  <xacro:property name="M_PI" value="3.1415926535897931"/>
+  <!-- <xacro:include filename="$(find plug_description)/urdf/wheelbase.urdf.xacro" />
   <xacro:wheeler_base_macro>
     <origin xyz="$(arg origin_xyz)" rpy="$(arg origin_rpy)"/>
@@ -14,5 +15,6 @@
     <xacro:property name="base_z" value="0.125" />
     <xacro:property name="bumper_z" value="0.175" />
-  </xacro:wheeler_base_macro>
+  </xacro:wheeler_base_macro> -->
+  <link name="world"/>
   <!--iiwa14-->
   <!-- Import Rviz colors -->
@@ -20,19 +22,20 @@
   <!--Import the lbr iiwa macro -->
   <xacro:include filename="$(find iiwa_description)/urdf/iiwa14.xacro"/>
-  <xacro:iiwa14 hardware_interface="$(arg hardware_interface)" robot_name="$(arg robot_name)" parent="link_base">
-    <origin xyz="0 0 0.125" rpy="0 0 0" />
+  <xacro:iiwa14 hardware_interface="$(arg hardware_interface)" robot_name="$(arg robot_name)" parent="world">
+    <!-- <origin xyz="0 0 0.125" rpy="0 0 0" /> -->
+    <origin xyz="$(arg origin_xyz)" rpy="$(arg origin_rpy)"/>
   </xacro:iiwa14>
   <!--plug-->
   <xacro:include filename="$(find plug_description)/urdf/plug.urdf.xacro"/>
   <xacro:plug parent="iiwa_link_ee">
-    <origin xyz="-0.011 -0.011 0.005" rpy="0 0 1.57" />
+    <origin xyz="-0.011 -0.011 0.005" rpy="0 0 ${M_PI/2}" />
   </xacro:plug>
   <!--camera-->
   <xacro:include filename="$(find plug_description)/urdf/camera.urdf.xacro"/>
   <xacro:rpi parent="iiwa_link_ee">
-    <origin xyz="-0.01 0 0.062" rpy="0 -1.57 0" />
+    <origin xyz="-0.015 0 0.062" rpy="0 ${-M_PI/2} 0" />
   </xacro:rpi>
   <!--RGB-D camera, look forward-->
-  <xacro:include filename="$(find plug_description)/urdf/realsense.urdf.xacro" />
+  <!-- <xacro:include filename="$(find plug_description)/urdf/realsense.urdf.xacro" />
   <xacro:realsense_macro parent="link_fbumper">
     <xacro:property name="location_x" value="0.05"/>
@@ -42,4 +45,4 @@
     <xacro:property name="camera_height" value="480" />
     <xacro:property name="camera_name" value="rs435" />
-  </xacro:realsense_macro>
+  </xacro:realsense_macro> -->
 </robot>

File: plug_description/urdf/plug.urdf.xacro (robot description, xacro)
@@ -2,4 +2,5 @@
 <robot xmlns:xacro="https://www.ros.org/wiki/xacro" >
   <xacro:property name="plug_m" value="0.1"/>
+  <xacro:property name="M_PI" value="3.1415926535897931"/>
   <xacro:macro name="plug" params="parent *origin">
     <!--plug-->
@@ -50,4 +51,37 @@
       </inertial>
     </link>
+    <joint name="joint_bumper" type="fixed">
+      <origin xyz="0.011 -0.013 0.0705" rpy="0 ${M_PI/2} 0"/>
+      <parent link="link_plug"/>
+      <child link="link_bumper"/>
+    </joint>
+    <link name="link_bumper">
+      <visual>
+        <origin xyz="0 0 0" rpy="0 0 0"/>
+        <geometry>
+          <box size="0.001 0.002 0.005"/>
+        </geometry>
+      </visual>
+      <collision name="bump_sensor_collision">
+        <origin xyz="0 0 0" rpy="0 0 0"/>
+        <geometry>
+          <box size="0.001 0.002 0.005"/>
+        </geometry>
+      </collision>
+    </link>
+    <gazebo reference="link_bumper">
+      <material>Gazebo/Blue</material>
+      <sensor name="main_bumper" type="contact">
+        <contact>
+          <collision>link_plug_base_fixed_joint_lump__bump_sensor_collision_collision_2</collision>
+        </contact>
+        <plugin name="gazebo_ros_bumper_controller" filename="libgazebo_ros_bumper.so">
+          <bumperTopicName>bumper_plug</bumperTopicName>
+          <frameName>world</frameName>
+          <alwaysOn>true</alwaysOn>
+          <updateRate>5.0</updateRate>
+        </plugin>
+      </sensor>
+    </gazebo>
   </xacro:macro>
 </robot>

Commit message: add depth sensor

File: plug_description/urdf/mmrobot.urdf.xacro (robot description, xacro)
@@ -22,4 +22,5 @@
   <!--Import the lbr iiwa macro -->
   <xacro:include filename="$(find iiwa_description)/urdf/iiwa14.xacro"/>
+  <!-- <xacro:iiwa14 hardware_interface="$(arg hardware_interface)" robot_name="$(arg robot_name)" parent="link_base"> -->
   <xacro:iiwa14 hardware_interface="$(arg hardware_interface)" robot_name="$(arg robot_name)" parent="world">
     <!-- <origin xyz="0 0 0.125" rpy="0 0 0" /> -->
@@ -39,7 +40,5 @@
   <!-- <xacro:include filename="$(find plug_description)/urdf/realsense.urdf.xacro" />
   <xacro:realsense_macro parent="link_fbumper">
-    <xacro:property name="location_x" value="0.05"/>
-    <xacro:property name="location_y" value="0.0"/>
-    <xacro:property name="location_z" value="0.07"/>
+    <origin xyz="0.0608 0 0.07" rpy="0 0 0" />
     <xacro:property name="camera_width" value="640" />
     <xacro:property name="camera_height" value="480" />

File: plug_description/urdf/realsense.urdf.xacro (robot description, xacro)
@@ -2,7 +2,4 @@
 <robot xmlns:xacro="https://www.ros.org/wiki/xacro" >
     <xacro:property name="M_PI" value="3.1415926535897931"/>
-    <xacro:property name="location_x" value="0" />
-    <xacro:property name="location_y" value="0" />
-    <xacro:property name="location_z" value="1.0" />
     <xacro:property name="realsense_d435_width" value="0.09"/>
     <xacro:property name="realsense_d435_height" value="0.025"/>
@@ -19,8 +16,8 @@
     <xacro:property name="camera_height" value="480" />
     <xacro:property name="camera_name" value="rs435" />
-    <xacro:macro name="realsense_macro" params="parent">
+    <xacro:macro name="realsense_macro" params="parent *origin">
       <!--camera-->
       <joint name="joint_rs435" type="fixed">
-        <origin xyz="${location_x+realsense_d435_depth/2.0} ${location_y} ${location_z}" rpy="0 0 0"/>
+        <xacro:insert_block name="origin"/>
         <parent link="${parent}"/>
         <child link="link_rs435"/>

Commit message: add ddpg

File: plug_description/urdf/mmrobot.urdf.xacro (robot description, xacro)
@@ -35,10 +35,10 @@
   <xacro:include filename="$(find plug_description)/urdf/camera.urdf.xacro"/>
   <xacro:rpi parent="iiwa_link_ee">
-    <origin xyz="-0.015 0 0.062" rpy="0 ${-M_PI/2} 0" />
+    <origin xyz="-0.06 0 0.02" rpy="0 ${-M_PI/2} 0" />
   </xacro:rpi>
   <!--RGB-D camera, look forward-->
   <!-- <xacro:include filename="$(find plug_description)/urdf/realsense.urdf.xacro" />
-  <xacro:realsense_macro parent="link_fbumper">
-    <origin xyz="0.0608 0 0.07" rpy="0 0 0" />
+  <xacro:realsense_macro parent="iiwa_link_ee">
+    <origin xyz="-0.06 0 0.02" rpy="0 ${-M_PI/2} 0" />
     <xacro:property name="camera_width" value="640" />
     <xacro:property name="camera_height" value="480" />

File: plug_description/urdf/realsense.urdf.xacro (robot description, xacro)
@@ -32,5 +32,5 @@
           <origin xyz="${realsense_d435_front_to_depth} ${realsense_d435_case_offset_y} 0.0" rpy="${M_PI/2} 0 ${M_PI/2}" />
           <geometry>
-            <mesh filename="package://ids_description/meshes/camera/D435.dae" scale="0.001 0.001 0.001" />
+            <mesh filename="package://plug_gazebo/media/materials/dae/D435.dae" scale="0.001 0.001 0.001" />
           </geometry>
         </visual>
@@ -46,5 +46,5 @@
         <material>Gazebo/Grey</material>
         <sensor type="depth" name="rs435">
-          <update_rate>30</update_rate>
+          <update_rate>30.0</update_rate>
           <camera>
             <horizontal_fov>${69.4*M_PI/180.0}</horizontal_fov>
@@ -52,5 +52,5 @@
             <diagonal_fov>${77.0*M_PI/180.0}</diagonal_fov>
             <image>
-              <format>B8G8R8</format>
+              <format>R8G8B8</format>
               <width>${camera_width}</width>
               <height>${camera_height}</height>
@@ -60,6 +60,14 @@
               <far>9.0</far>
             </clip>
+            <noise>
+              <type>gaussian</type>
+              <mean>0.0</mean>
+              <stddev>0.007</stddev>
+            </noise>
           </camera>
           <plugin name="rs435_camera_plugin" filename="libgazebo_ros_openni_kinect.so">
+            <baseline>0.2</baseline>
+            <alwaysOn>true</alwaysOn>
+            <updateRate>1.0</updateRate>
             <cameraName>${camera_name}</cameraName>
             <imageTopicName>color/image_raw</imageTopicName>
@@ -69,4 +77,16 @@
             <pointCloudTopicName>depth/points</pointCloudTopicName>
             <frameName>rs435_frame</frameName>
+            <pointCloudCutoff>0.5</pointCloudCutoff>
+            <pointCloudCutoffMax>3.0</pointCloudCutoffMax>
+            <distortionK1>0.00000001</distortionK1>
+            <distortionK2>0.00000001</distortionK2>
+            <distortionK3>0.00000001</distortionK3>
+            <distortionT1>0.00000001</distortionT1>
+            <distortionT2>0.00000001</distortionT2>
+            <CxPrime>0</CxPrime>
+            <Cx>0</Cx>
+            <Cy>0</Cy>
+            <focalLength>0</focalLength>
+            <hackBaseline>0</hackBaseline>
           </plugin>
         </sensor>
